File: _debugger/black_magic_probe/rp_pico_bmp_probe.kicad_pcb (KiCad board)
At the start: 2 copper layers, 51.5 x 67.7 mm, 13 parts, among them J1 Conn_01x03_Pin, J2 Conn_01x04_Pin, J3 Conn_01x02_Pin, J4 Conn_01x02_Pin

Commit message: Added readme
Other:
- board text added: "3V3"
- board text added: "GND"
- board text added: "RX"
- board text added: "SWCLK"
- board text added: "SWIO"
- board text added: "TDI"
- board text added: "TDO"
- board text added: "TX"
- board text added: "nRST"
Changed lines of the file:
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@@
 		(tags "connector Molex KK-254 vertical")
 		(property "Reference" "J4"
-			(at 1.27 -4.12 0)
+			(at 1.27 3.99 0)
 			(layer "F.SilkS")
 			(effects
@@
 		(tags "connector Molex KK-254 vertical")
 		(property "Reference" "J2"
-			(at 3.81 -4.12 0)
+			(at 3.81 4.25 0)
 			(layer "F.SilkS")
 			(effects
@@
 		(tags "connector Molex KK-254 vertical")
 		(property "Reference" "J1"
-			(at 2.54 -4.12 0)
+			(at 2.54 4.36 0)
 			(layer "F.SilkS")
 			(effects
@@
 		(tags "connector Molex KK-254 vertical")
 		(property "Reference" "J3"
-			(at 1.27 -4.12 0)
+			(at 1.27 3.96 0)
 			(layer "F.SilkS")
 			(effects
@@
 		(layer "Edge.Cuts")
 	)
+	(gr_text "TDO"
+		(at 98.4 105.1 90)
+		(layer "F.SilkS")
+		(effects
+			(font
+				(size 1 1)
+				(thickness 0.15)
+			)
+			(justify left bottom)
+		)
+	)
+	(gr_text "TDI"
+		(at 101.6 104.6 90)
+		(layer "F.SilkS")
+		(effects
+			(font
+				(size 1 1)
+				(thickness 0.15)
+			)
+			(justify left bottom)
+		)
+	)
+	(gr_text "GND"
+		(at 106.7 105.5 90)
+		(layer "F.SilkS")
+		(effects
+			(font
+				(size 1 1)
+				(thickness 0.15)
+			)
+			(justify left bottom)
+		)
+	)
+	(gr_text "3V3"
+		(at 110.1 104.9 90)
+		(layer "F.SilkS")
+		(effects
+			(font
+				(size 1 1)
+				(thickness 0.15)
+			)
+			(justify left bottom)
+		)
+	)
+	(gr_text "GND"
+		(at 114.4 105.2 90)
+		(layer "F.SilkS")
+		(effects
+			(font
+				(size 1 1)
+				(thickness 0.15)
+			)
+			(justify left bottom)
+		)
+	)
+	(gr_text "SWIO"
+		(at 116.8 104.7 90)
+		(layer "F.SilkS")
+		(effects
+			(font
+				(size 1 1)
+				(thickness 0.15)
+			)
+			(justify left bottom)
+		)
+	)
+	(gr_text "SWCLK"
+		(at 119.3 105 90)
+		(layer "F.SilkS")
+		(effects
+			(font
+				(size 1 1)
+				(thickness 0.15)
+			)
+			(justify left bottom)
+		)
+	)
+	(gr_text "nRST"
+		(at 121.81 104.89 90)
+		(layer "F.SilkS")
+		(effects
+			(font
+				(size 1 1)
+				(thickness 0.15)
+			)
+			(justify left bottom)
+		)
+	)
+	(gr_text "GND"
+		(at 128 105.13 90)
+		(layer "F.SilkS")
+		(effects
+			(font
+				(size 1 1)
+				(thickness 0.15)
+			)
+			(justify left bottom)
+		)
+	)
+	(gr_text "RX"
+		(at 130.66 105.13 90)
+		(layer "F.SilkS")
+		(effects
+			(font
+				(size 1 1)
+				(thickness 0.15)
+			)
+			(justify left bottom)
+		)
+	)
+	(gr_text "TX"
+		(at 133.2 105.24 90)
+		(layer "F.SilkS")
+		(effects
+			(font
+				(size 1 1)
+				(thickness 0.15)
+			)
+			(justify left bottom)
+		)
+	)
 	(segment
 		(start 123.05 75)
@@
 		)
 		(min_thickness 0.25)
-		(fill yes
+		(fill
 			(thermal_gap 0.5)
 			(thermal_bridge_width 0.5)
